File: KiCAD/Garage Door Opener/Garage Door Opener.kicad_pcb (KiCad board)
At the start: 2 copper layers, 57 x 57 mm, 10 parts, among them J1 Screw_Terminal_01x03, J3 Conn_01x02_Pin, K1 JQC-3FF-S-Z, Q1 S8550, SW1 SW_Push_Dual, U1 YD-ESP32-S3

Commit message: Updated board design
Parts:
- removed REF** (x2): MountingHole_2.5mm, MountingHole:MountingHole_2.5mm
- added H1: MountingHole, MountingHole:MountingHole_3.5mm, F.Cu at (67.8, 54.8)
- added H2: MountingHole, MountingHole:MountingHole_3.5mm, F.Cu at (117.2, 54.8)
- Q1: value S8550 -> PN2222A; footprint Package_TO_SOT_SMD:SOT-23 -> Package_TO_SOT_THT:TO-92_Inline
- SW1: value SW_Push_Dual -> SW_Push
- moved D1 24.7 mm to (106.5, 72.1)
- moved Q1 22.4 mm to (107.3, 64.4), turned to -90 degrees
- moved R1 18.7 mm to (102.0, 65.6), turned to 0 degrees
- moved J3 7.57 mm to (107.6, 57.3), turned to -90 degrees
- moved SW1 0.95 mm to (115.3, 66.3)
Connections:
- D1 pad 1: Net-(D1-K) -> +5V
- D1 pad 2: GND -> Net-(D1-A)
- J3 pad 1: Net-(J3-Pin_1) -> GND
- J3 pad 2: GND -> Net-(J3-Pin_2)
- K1 pad 1: Net-(D1-K) -> +5V
- K1 pad 2: GND -> Net-(D1-A)
- Q1 pad 1: Net-(Q1-E) -> GND
- Q1 pad 2: +5V -> Net-(Q1-B)
- Q1 pad 3: Net-(D1-K) -> Net-(D1-A)
- R1 pad 1: Net-(U1-GPIO5/ADC1_CH4) -> Net-(U1-GPIO11/ADC2_CH0)
- R1 pad 2: Net-(Q1-E) -> Net-(Q1-B)
- SW1 pad 1: +5V -> Net-(D1-A)
- SW1 pad 2: Net-(D1-K) -> GND
- U1 pad 17: unconnected-(U1-GPIO11/ADC2_CH0-Pad17) -> Net-(U1-GPIO11/ADC2_CH0)
- U1 pad 18: unconnected-(U1-GPIO12/ADC2_CH1-Pad18) -> Net-(J3-Pin_2)
- U1 pad 5: Net-(U1-GPIO5/ADC1_CH4) -> unconnected-(U1-GPIO5/ADC1_CH4-Pad5)
- U1 pad 6: Net-(J3-Pin_1) -> unconnected-(U1-GPIO6/ADC1_CH5-Pad6)
Routing:
- net Net-(D1-K): track 69.6 -> 0.00 mm, vias 2 -> 0
- net Net-(U1-GPIO5/ADC1_CH4): track 35.7 -> 0.00 mm
- net Net-(J3-Pin_1): track 32.7 -> 0.00 mm
- net Net-(D1-A): track 0.00 -> 24.4 mm
- net Net-(J3-Pin_2): track 0.00 -> 9.70 mm
- net +5V: track 45.2 -> 40.5 mm, vias 0 -> 2
- net Net-(Q1-B): track 0.00 -> 4.39 mm
- net Net-(Q1-E): track 3.75 -> 0.00 mm
- net Net-(U1-GPIO11/ADC2_CH0): track 0.00 -> 3.36 mm
- net /Normally Open: track 10.6 -> 12.1 mm
- net unconnected-(U1-GPIO6/ADC1_CH5-Pad6): track 0.00 -> 0.78 mm
- added copper zone on B.Cu, net GND
Other:
- board text added: "chrisdaun@gmail.com Garage Door Opener v2.0"
- board text removed: "chrisdaun@gmail.com Garage Door Opener v1.0"
